File: PCB/dETECTOR DE INCENDIO/ControlRele.kicad_sch (KiCad schematic)
At the start: 4 parts, among them K4 FINDER-36.11, Q1 PN2222A

Commit message: Se crea dise;o preliminar de PCB
Parts:
- removed Q1: PN2222A, Package_TO_SOT_THT:TO-92_Inline, symbol Transistor_BJT:PN2222A
- added Q3: BCX56, Package_TO_SOT_SMD:SOT-89-3, symbol Transistor_BJT:BCX56
- renumbered D1 to D4
Connections:
- net GND: now also Q3.3 (E)
- net at R4.2: now also Q3.1 (B)
- net at D4.2 (A), K4.A2: now also Q3.2 (C)
Changed lines of the file:
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@@
     (effects (font (size 1.27 1.27)) (justify left))
   )
-  (symbol (lib_id "Transistor_BJT:PN2222A") (at 138.43 96.52 0) (unit 1)
+  (symbol (lib_id "Transistor_BJT:BCX56") (at 138.43 96.52 0) (unit 1)
     (in_bom yes) (on_board yes) (dnp no) (fields_autoplaced)
-    (property "Reference" "Q1" (at 143.51 95.885 0)
+    (property "Reference" "Q3" (at 143.51 95.25 0)
       (effects (font (size 1.27 1.27)) (justify left))
     )
-    (property "Value" "PN2222A" (at 143.51 98.425 0)
+    (property "Value" "BCX56" (at 143.51 97.79 0)
       (effects (font (size 1.27 1.27)) (justify left))
     )
-    (property "Footprint" "Package_TO_SOT_THT:TO-92_Inline" (at 143.51 98.425 0)
+    (property "Footprint" "Package_TO_SOT_SMD:SOT-89-3" (at 143.51 98.425 0)
       (effects (font (size 1.27 1.27) italic) (justify left) hide)
     )
-    (property "Datasheet" "https://www.onsemi.com/pub/Collateral/PN2222-D.PDF" (at 138.43 96.52 0)
+    (property "Datasheet" "https://www.nxp.com/docs/en/data-sheet/BCP56_BCX56_BC56PA.pdf" (at 138.43 96.52 0)
       (effects (font (size 1.27 1.27)) (justify left) hide)
     )
+    (pin "3")
     (pin "1")
     (pin "2")
-    (pin "3")
     (instances
       (project "dETECTOR DE INCENDIO"
-        (path "/891e9ece-129f-48de-add1-9005b83b8618/8fe89136-e154-4bbc-a8e2-8037deb6ac66"
-          (reference "Q1") (unit 1)
-        )
         (path "/891e9ece-129f-48de-add1-9005b83b8618/d4fd6b5d-3307-47ad-9bfb-dcbb01c2f688"
-          (reference "Q1") (unit 1)
+          (reference "Q3") (unit 1)
         )
         (path "/891e9ece-129f-48de-add1-9005b83b8618/961c37f3-fc98-4450-9285-f1cd0c0b2006"
-          (reference "Q2") (unit 1)
+          (reference "Q4") (unit 1)
         )
       )
@@
     (instances
       (project "dETECTOR DE INCENDIO"
-        (path "/891e9ece-129f-48de-add1-9005b83b8618/8fe89136-e154-4bbc-a8e2-8037deb6ac66"
-          (reference "R4") (unit 1)
-        )
         (path "/891e9ece-129f-48de-add1-9005b83b8618/d4fd6b5d-3307-47ad-9bfb-dcbb01c2f688"
           (reference "R4") (unit 1)
@@
   (symbol (lib_id "Diode:SM4007") (at 140.97 85.09 270) (unit 1)
     (in_bom yes) (on_board yes) (dnp no) (fields_autoplaced)
-    (property "Reference" "D1" (at 143.51 84.455 90)
+    (property "Reference" "D4" (at 143.51 84.455 90)
       (effects (font (size 1.27 1.27)) (justify left))
     )
@@
     (instances
       (project "dETECTOR DE INCENDIO"
-        (path "/891e9ece-129f-48de-add1-9005b83b8618/db2f7c0d-1a4e-4a60-ac10-5a37332c5708"
-          (reference "D1") (unit 1)
-        )
-        (path "/891e9ece-129f-48de-add1-9005b83b8618/8fe89136-e154-4bbc-a8e2-8037deb6ac66"
-          (reference "D4") (unit 1)
-        )
         (path "/891e9ece-129f-48de-add1-9005b83b8618/d4fd6b5d-3307-47ad-9bfb-dcbb01c2f688"
           (reference "D4") (unit 1)
