File: PCB/dETECTOR DE INCENDIO/MCU.kicad_sch (KiCad schematic)
At the start: 6 parts

Commit message: Se crea dise;o preliminar de PCB
Connections:
- net BocinaEmergencia: now also MOD1.11 (GPIO38); no longer MOD1.33 (GPIO20)
- net Calidad: now also MOD1.3 (GPIO12); no longer MOD1.18 (GPIO01)
- net DHT: now also MOD1.33 (GPIO20); no longer MOD1.26 (GPIO16)
- net LED1: now also R2.1; no longer R1.1
- net LED2: now also R1.1; no longer R2.1
- net Lampara: now also MOD1.12 (GPIO39); no longer MOD1.34 (GPIO26)
Changed lines of the file:
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@@
-    (stroke (width 0) (type default))
-  )
-  (wire (pts (xy 148.59 88.9) (xy 152.4 88.9))
     (stroke (width 0) (type default))
   )
@@
     (stroke (width 0) (type default))
   )
-  (wire (pts (xy 148.59 96.52) (xy 152.4 96.52))
+  (wire (pts (xy 148.59 96.52) (xy 153.67 96.52))
+    (stroke (width 0) (type default))
+  )
+  (wire (pts (xy 120.65 83.82) (xy 123.19 83.82))
+    (stroke (width 0) (type default))
+  )
+  (wire (pts (xy 119.38 60.96) (xy 123.19 60.96))
     (stroke (width 0) (type default))
   )
@@
     (stroke (width 0) (type default))
   )
+  (wire (pts (xy 148.59 91.44) (xy 151.13 91.44))
+    (stroke (width 0) (type default))
+  )
   (wire (pts (xy 148.59 81.28) (xy 153.67 81.28))
     (stroke (width 0) (type default))
@@
   )
   (wire (pts (xy 148.59 101.6) (xy 152.4 101.6))
+    (stroke (width 0) (type default))
+  )
+  (wire (pts (xy 148.59 93.98) (xy 151.13 93.98))
     (stroke (width 0) (type default))
   )
@@
     (stroke (width 0) (type default))
   )
-  (wire (pts (xy 119.38 99.06) (xy 123.19 99.06))
-    (stroke (width 0) (type default))
-  )
   (wire (pts (xy 148.59 71.12) (xy 153.67 71.12))
     (stroke (width 0) (type default))
@@
     (stroke (width 0) (type default))
   )
-  (wire (pts (xy 148.59 68.58) (xy 152.4 68.58))
+  (wire (pts (xy 120.65 81.28) (xy 123.19 81.28))
     (stroke (width 0) (type default))
   )
@@
     (effects (font (size 1.27 1.27)) (justify left bottom))
   )
+  (label "LED2" (at 236.22 53.34 180) (fields_autoplaced)
+    (effects (font (size 1.27 1.27)) (justify right bottom))
+  )
   (label "Buzzer" (at 242.57 25.4 0) (fields_autoplaced)
     (effects (font (size 1.27 1.27)) (justify left bottom))
-  )
-  (label "LED1" (at 236.22 53.34 180) (fields_autoplaced)
-    (effects (font (size 1.27 1.27)) (justify right bottom))
   )
   (label "LED2" (at 152.4 63.5 0) (fields_autoplaced)
     (effects (font (size 1.27 1.27)) (justify left bottom))
   )
-  (label "LED2" (at 236.22 60.96 180) (fields_autoplaced)
-    (effects (font (size 1.27 1.27)) (justify right bottom))
-  )
   (label "LED3" (at 236.22 68.58 180) (fields_autoplaced)
     (effects (font (size 1.27 1.27)) (justify right bottom))
   )
-  (label "Buzzer" (at 152.4 96.52 0) (fields_autoplaced)
+  (label "LED1" (at 236.22 60.96 180) (fields_autoplaced)
+    (effects (font (size 1.27 1.27)) (justify right bottom))
+  )
+  (label "Buzzer" (at 153.67 96.52 0) (fields_autoplaced)
     (effects (font (size 1.27 1.27)) (justify left bottom))
   )
@@
     (effects (font (size 1.27 1.27)) (justify left))
   )
-  (hierarchical_label "Calidad" (shape input) (at 119.38 99.06 180) (fields_autoplaced)
-    (effects (font (size 1.27 1.27)) (justify right))
-  )
-  (hierarchical_label "Lampara" (shape input) (at 152.4 68.58 0) (fields_autoplaced)
-    (effects (font (size 1.27 1.27)) (justify left))
-  )
   (hierarchical_label "CLK" (shape input) (at 120.65 76.2 180) (fields_autoplaced)
     (effects (font (size 1.27 1.27)) (justify right))
-  )
-  (hierarchical_label "BocinaEmergencia" (shape input) (at 153.67 71.12 0) (fields_autoplaced)
-    (effects (font (size 1.27 1.27)) (justify left))
   )
   (hierarchical_label "GND" (shape input) (at 274.32 60.96 0) (fields_autoplaced)
@@
     (effects (font (size 1.27 1.27)) (justify left))
   )
+  (hierarchical_label "BocinaEmergencia" (shape input) (at 120.65 81.28 180) (fields_autoplaced)
+    (effects (font (size 1.27 1.27)) (justify right))
+  )
+  (hierarchical_label "Calidad" (shape input) (at 119.38 60.96 180) (fields_autoplaced)
+    (effects (font (size 1.27 1.27)) (justify right))
+  )
+  (hierarchical_label "Lampara" (shape input) (at 120.65 83.82 180) (fields_autoplaced)
+    (effects (font (size 1.27 1.27)) (justify right))
+  )
   (hierarchical_label "CS" (shape input) (at 120.65 73.66 180) (fields_autoplaced)
     (effects (font (size 1.27 1.27)) (justify right))
@@
     (effects (font (size 1.27 1.27)) (justify right))
   )
-  (hierarchical_label "DHT" (shape bidirectional) (at 152.4 88.9 0) (fields_autoplaced)
-    (effects (font (size 1.27 1.27)) (justify left))
-  )
   (hierarchical_label "GND" (shape input) (at 135.89 113.03 270) (fields_autoplaced)
     (effects (font (size 1.27 1.27)) (justify right))
   )
+  (hierarchical_label "DHT" (shape bidirectional) (at 153.67 71.12 0) (fields_autoplaced)
+    (effects (font (size 1.27 1.27)) (justify left))
+  )
   (hierarchical_label "Trigger" (shape output) (at 152.4 101.6 0) (fields_autoplaced)
