File: PCB/dETECTOR DE INCENDIO/Regulador_de_voltaje.kicad_sch (KiCad schematic)
At the start: 6 parts, among them U1 AMS1117-3.3

Commit message: Se crea dise;o preliminar de PCB
Parts:
- removed D1, D3: SM4007, Diode_SMD:D_MELF, symbol Diode:SM4007
- removed PS1: HLK-10M05, Converter_ACDC:Converter_ACDC_HiLink_HLK-10Mxx, symbol Converter_ACDC:HLK-10M05
- added PS2: HLK-20M05, Converter_ACDC:Converter_ACDC_Hi-Link_HLK-20Mxx, symbol Converter_ACDC:HLK-20M05
Connections:
- net +5v: now also C2.1, U1.3 (VI), PS2.4 (+Vout)
- net GND: now also PS2.3 (-Vout)
- net L: now also PS2.1 (AC/L)
- net N: now also PS2.2 (AC/N)
Changed lines of the file:
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@@
   (junction (at 138.43 63.5) (diameter 0) (color 0 0 0 0)
-  )
-  (junction (at 127 43.18) (diameter 0) (color 0 0 0 0)
   )
   (junction (at 149.86 48.26) (diameter 0) (color 0 0 0 0)
@@
   (junction (at 138.43 59.69) (diameter 0) (color 0 0 0 0)
   )
-  (wire (pts (xy 111.76 35.56) (xy 127 35.56))
-    (stroke (width 0) (type default))
-  )
-  (wire (pts (xy 127 43.18) (xy 127 48.26))
+  (wire (pts (xy 125.73 46.99) (xy 125.73 48.26))
     (stroke (width 0) (type default))
   )
@@
     (stroke (width 0) (type default))
   )
-  (wire (pts (xy 111.76 43.18) (xy 127 43.18))
-    (stroke (width 0) (type default))
-  )
   (wire (pts (xy 48.26 36.83) (xy 55.88 36.83))
     (stroke (width 0) (type default))
   )
   (wire (pts (xy 138.43 59.69) (xy 138.43 55.88))
-    (stroke (width 0) (type default))
-  )
-  (wire (pts (xy 102.87 35.56) (xy 104.14 35.56))
     (stroke (width 0) (type default))
   )
@@
     (stroke (width 0) (type default))
   )
-  (wire (pts (xy 127 35.56) (xy 127 43.18))
+  (wire (pts (xy 125.73 48.26) (xy 127 48.26))
     (stroke (width 0) (type default))
   )
@@
     (stroke (width 0) (type default))
   )
-  (wire (pts (xy 102.87 43.18) (xy 104.14 43.18))
-    (stroke (width 0) (type default))
-  )
   (wire (pts (xy 152.4 48.26) (xy 149.86 48.26))
     (stroke (width 0) (type default))
@@
     (stroke (width 0) (type default))
   )
-  (hierarchical_label "Vbat" (shape input) (at 102.87 43.18 180) (fields_autoplaced)
-    (effects (font (size 1.27 1.27)) (justify right))
-  )
-  (hierarchical_label "+5v" (shape output) (at 102.87 35.56 180) (fields_autoplaced)
-    (effects (font (size 1.27 1.27)) (justify right))
+  (hierarchical_label "+5v" (shape output) (at 125.73 46.99 90) (fields_autoplaced)
+    (effects (font (size 1.27 1.27)) (justify left))
   )
   (hierarchical_label "GND" (shape output) (at 139.7 63.5 0) (fields_autoplaced)
@@
     (effects (font (size 1.27 1.27)) (justify right))
   )
-  (symbol (lib_id "Diode:SM4007") (at 107.95 35.56 180) (unit 1)
-    (in_bom yes) (on_board yes) (dnp no) (fields_autoplaced)
-    (property "Reference" "D1" (at 107.95 30.48 0)
-      (effects (font (size 1.27 1.27)))
-    )
-    (property "Value" "SM4007" (at 107.95 33.02 0)
-      (effects (font (size 1.27 1.27)))
-    )
-    (property "Footprint" "Diode_SMD:D_MELF" (at 107.95 31.115 0)
-      (effects (font (size 1.27 1.27)) hide)
-    )
-    (property "Datasheet" "http://cdn-reichelt.de/documents/datenblatt/A400/SMD1N400%23DIO.pdf" (at 107.95 35.56 0)
-      (effects (font (size 1.27 1.27)) hide)
-    )
-    (property "Sim.Device" "D" (at 107.95 35.56 0)
-      (effects (font (size 1.27 1.27)) hide)
-    )
-    (property "Sim.Pins" "1=K 2=A" (at 107.95 35.56 0)
-      (effects (font (size 1.27 1.27)) hide)
-    )
-    (pin "1")
-    (pin "2")
-    (instances
-      (project "dETECTOR DE INCENDIO"
-        (path "/891e9ece-129f-48de-add1-9005b83b8618/db2f7c0d-1a4e-4a60-ac10-5a37332c5708"
-          (reference "D1") (unit 1)
-        )
-      )
-    )
-  )
-  (symbol (lib_id "Diode:SM4007") (at 107.95 43.18 180) (unit 1)
-    (in_bom yes) (on_board yes) (dnp no)
-    (property "Reference" "D3" (at 107.95 38.1 0)
-      (effects (font (size 1.27 1.27)))
-    )
-    (property "Value" "SM4007" (at 107.95 40.64 0)
-      (effects (font (size 1.27 1.27)))
-    )
-    (property "Footprint" "Diode_SMD:D_MELF" (at 107.95 38.735 0)
-      (effects (font (size 1.27 1.27)) hide)
-    )
-    (property "Datasheet" "http://cdn-reichelt.de/documents/datenblatt/A400/SMD1N400%23DIO.pdf" (at 107.95 43.18 0)
-      (effects (font (size 1.27 1.27)) hide)
-    )
-    (property "Sim.Device" "D" (at 107.95 43.18 0)
-      (effects (font (size 1.27 1.27)) hide)
-    )
-    (property "Sim.Pins" "1=K 2=A" (at 107.95 43.18 0)
-      (effects (font (size 1.27 1.27)) hide)
-    )
-    (pin "1")
-    (pin "2")
-    (instances
-      (project "dETECTOR DE INCENDIO"
-        (path "/891e9ece-129f-48de-add1-9005b83b8618/db2f7c0d-1a4e-4a60-ac10-5a37332c5708"
-          (reference "D3") (unit 1)
-        )
-      )
-    )
-  )
   (symbol (lib_id "Regulator_Linear:AMS1117-3.3") (at 138.43 48.26 0) (unit 1)
     (in_bom yes) (on_board yes) (dnp no) (fields_autoplaced)
@@
     (instances
       (project "dETECTOR DE INCENDIO"
-        (path "/891e9ece-129f-48de-add1-9005b83b8618"
-          (reference "U1") (unit 1)
-        )
         (path "/891e9ece-129f-48de-add1-9005b83b8618/db2f7c0d-1a4e-4a60-ac10-5a37332c5708"
           (reference "U1") (unit 1)
@@
     )
   )
-  (symbol (lib_id "Converter_ACDC:HLK-10M05") (at 66.04 39.37 0) (unit 1)
+  (symbol (lib_id "Converter_ACDC:HLK-20M05") (at 66.04 39.37 0) (unit 1)
     (in_bom yes) (on_board yes) (dnp no) (fields_autoplaced)
-    (property "Reference" "PS1" (at 66.04 31.75 0)
+    (property "Reference" "PS2" (at 66.04 30.48 0)
       (effects (font (size 1.27 1.27)))
     )
-    (property "Value" "HLK-10M05" (at 66.04 34.29 0)
+    (property "Value" "HLK-20M05" (at 66.04 33.02 0)
       (effects (font (size 1.27 1.27)))
     )
-    (property "Footprint" "Converter_ACDC:Converter_ACDC_HiLink_HLK-10Mxx" (at 66.04 46.355 0)
+    (property "Footprint" "Converter_ACDC:Converter_ACDC_Hi-Link_HLK-20Mxx" (at 66.04 46.355 0)
       (effects (font (size 1.27 1.27)) hide)
     )
-    (property "Datasheet" "http://h.hlktech.com/download/ACDC%E7%94%B5%E6%BA%90%E6%A8%A1%E5%9D%9710W%E7%B3%BB%E5%88%97/1/%E6%B5%B7%E5%87%8C%E7%A7%9110W%E7%B3%BB%E5%88%97%E7%94%B5%E6%BA%90%E6%A8%A1%E5%9D%97%E8%A7%84%E6%A0%BC%E4%B9%A6V1.8.pdf" (at 66.04 48.26 0)
+    (property "Datasheet" "https://h.hlktech.com/download/ACDC%E7%94%B5%E6%BA%90%E6%A8%A1%E5%9D%9720W%E7%B3%BB%E5%88%97/1/%E6%B5%B7%E5%87%8C%E7%A7%9120W%E7%B3%BB%E5%88%97%E7%94%B5%E6%BA%90%E6%A8%A1%E5%9D%97%E8%A7%84%E6%A0%BC%E4%B9%A6V1.6.pdf" (at 66.04 48.26 0)
       (effects (font (size 1.27 1.27)) hide)
     )
+    (pin "3")
+    (pin "4")
     (pin "1")
     (pin "2")
-    (pin "3")
-    (pin "4")
     (instances
       (project "dETECTOR DE INCENDIO"
-        (path "/891e9ece-129f-48de-add1-9005b83b8618"
-          (reference "PS1") (unit 1)
-        )
         (path "/891e9ece-129f-48de-add1-9005b83b8618/db2f7c0d-1a4e-4a60-ac10-5a37332c5708"
-          (reference "PS1") (unit 1)
+          (reference "PS2") (unit 1)
         )
       )
