File: PCB/dETECTOR DE INCENDIO/Sensores.kicad_sch (KiCad schematic)
At the start: 5 parts, among them J10 Ultra Sonido, J11 GPS, J7 DHT11, J8 Sensor De Calidad De Aire, J9 Termocupla

Commit message: Se crea dise;o preliminar de PCB
Parts:
- removed J9: Termocupla, Connector_JST:JST_XH_B5B-XH-AM_1x05_P2.50mm_Vertical, symbol Connector_Generic:Conn_01x05
- added J5: Temp, Connector_JST:JST_XH_B5B-XH-A_1x05_P2.50mm_Vertical, symbol Connector_Generic:Conn_01x05
Connections:
- net +3.3v: now also J5.2 (Pin_2)
- net CS: now also J5.4 (Pin_4)
- net DO: now also J5.5 (Pin_5)
- net GND: now also J5.1 (Pin_1)
- net SCK: now also J5.3 (Pin_3)
Changed lines of the file:
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@@
   (symbol (lib_id "Connector_Generic:Conn_01x05") (at 161.29 107.95 0) (unit 1)
     (in_bom yes) (on_board yes) (dnp no) (fields_autoplaced)
-    (property "Reference" "J9" (at 163.83 107.315 0)
+    (property "Reference" "J5" (at 163.83 106.68 0)
       (effects (font (size 1.27 1.27)) (justify left))
     )
-    (property "Value" "Termocupla" (at 163.83 109.855 0)
+    (property "Value" "Temp" (at 163.83 109.22 0)
       (effects (font (size 1.27 1.27)) (justify left))
     )
-    (property "Footprint" "Connector_JST:JST_XH_B5B-XH-AM_1x05_P2.50mm_Vertical" (at 161.29 107.95 0)
+    (property "Footprint" "Connector_JST:JST_XH_B5B-XH-A_1x05_P2.50mm_Vertical" (at 161.29 107.95 0)
       (effects (font (size 1.27 1.27)) hide)
     )
@@
       (effects (font (size 1.27 1.27)) hide)
     )
+    (pin "4")
+    (pin "3")
+    (pin "2")
     (pin "1")
-    (pin "2")
-    (pin "3")
-    (pin "4")
     (pin "5")
     (instances
       (project "dETECTOR DE INCENDIO"
         (path "/891e9ece-129f-48de-add1-9005b83b8618/3aa8911b-3820-4dd0-b906-859df77c4344"
-          (reference "J9") (unit 1)
+          (reference "J5") (unit 1)
         )
       )
