File: PCB/dETECTOR DE INCENDIO/dETECTOR DE INCENDIO.kicad_pcb (KiCad board)
At the start: 2 copper layers, 28 parts, among them J1 Screw_Terminal_01x02, J10 Ultra Sonido, J11 GPS, J2 Conn_01x03, J3 Conn_01x03, J7 DHT11, J8 Sensor De Calidad De Aire, J9 Termocupla, K3 FINDER-36.11, K4 FINDER-36.11, Q1 PN2222A, Q2 PN2222A, U1 AMS1117-3.3

Commit message: Se crea dise;o preliminar de PCB
Parts:
- removed D1, D3: SM4007, Diode_SMD:D_MELF
- removed J9: Termocupla, Connector_JST:JST_XH_B5B-XH-AM_1x05_P2.50mm_Vertical
- removed PS1: HLK-10M05, Converter_ACDC:Converter_ACDC_HiLink_HLK-10Mxx
- removed Q1, Q2: PN2222A, Package_TO_SOT_THT:TO-92_Inline
- added J4: DHT11, Connector_JST:JST_XH_B3B-XH-A_1x03_P2.50mm_Vertical, F.Cu at (2.98, 2.88)
- added J5: Temp, Connector_JST:JST_XH_B5B-XH-A_1x05_P2.50mm_Vertical, F.Cu at (265.2, 104.3)
- added PS2: HLK-20M05, Converter_ACDC:Converter_ACDC_Hi-Link_HLK-20Mxx, F.Cu at (193.0, 60.9)
- added Q3: BCX56, Package_TO_SOT_SMD:SOT-89-3, F.Cu at (225.8, 103.1)
- added Q4: BCX56, Package_TO_SOT_SMD:SOT-89-3, F.Cu at (226.8, 131.6)
- moved BZ1 148.8 mm to (258.1, 138.9)
- moved J3 128.7 mm to (262.4, 121.0), turned to -90 degrees
- moved J2 122.9 mm to (259.4, 89.8), turned to -90 degrees
- moved C1 99.7 mm to (262.4, 64.0)
- moved J7 97.3 mm to (178.3, 119.0)
- moved D2 95.0 mm to (179.3, 138.9), turned to -90 degrees
- moved J10 93.1 mm to (179.1, 85.1), turned to -90 degrees
- moved J11 92.4 mm to (179.1, 99.3), turned to -90 degrees
- moved C2 92.0 mm to (256.3, 64.0)
- moved J8 90.2 mm to (178.5, 134.8)
- moved R2 86.9 mm to (187.5, 143.5), turned to 180 degrees
- moved U1 85.2 mm to (260.9, 72.9), turned to -90 degrees
- moved R1 81.3 mm to (187.5, 140.2), turned to 180 degrees
- moved R3 76.7 mm to (187.5, 137.2), turned to 180 degrees
- moved K4 75.7 mm to (234.2, 128.4), turned to 90 degrees
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Connections:
- C2 pad 1: Net-(D1-K) -> +5V
- J2 pad 2: /ControlRele1/NA -> /ControlRele1/COM
- J2 pad 3: /ControlRele1/COM -> /ControlRele1/NA
- J3 pad 2: /ControlRele2/NA -> /ControlRele2/COM
- J3 pad 3: /ControlRele2/COM -> /ControlRele2/NA
- MOD1 pad 11: unconnected-(MOD1-GPIO38-Pad11) -> /ControlRele1/Input
- MOD1 pad 12: unconnected-(MOD1-GPIO39-Pad12) -> /ControlRele2/Input
- MOD1 pad 18: /MCU/Calidad -> unconnected-(MOD1-GPIO01-Pad18)
- MOD1 pad 26: /MCU/DHT -> unconnected-(MOD1-GPIO16-Pad26)
- MOD1 pad 3: unconnected-(MOD1-GPIO12-Pad3) -> /MCU/Calidad
- MOD1 pad 33: /ControlRele2/Input -> /MCU/DHT
- MOD1 pad 34: /ControlRele1/Input -> unconnected-(MOD1-GPIO26-Pad34)
- R1 pad 1: /MCU/LED1 -> /MCU/LED2
- R2 pad 1: /MCU/LED2 -> /MCU/LED1
- U1 pad 3: Net-(D1-K) -> +5V
Routing:
- net GND: track 0.00 -> 452.2 mm
- net +3.3V: track 0.00 -> 244.1 mm
- net /MCU/Calidad: track 0.00 -> 137.6 mm
- net /MCU/Buzzer: track 0.00 -> 106.1 mm
- net +5V: track 0.00 -> 65.1 mm
- net /MCU/Do: track 0.00 -> 51.4 mm
- net /MCU/CS: track 0.00 -> 51.4 mm
- net /MCU/CLK: track 0.00 -> 51.3 mm
- net /ControlRele2/Input: track 0.00 -> 49.3 mm
- net /ControlRele2/COM: track 0.00 -> 31.5 mm
- net /ControlRele1/COM: track 0.00 -> 28.4 mm
- net Net-(D4-A): track 0.00 -> 28.0 mm
- net /MCU/TX1: track 0.00 -> 24.2 mm
- net Net-(D5-A): track 0.00 -> 24.2 mm
- net /MCU/LED1: track 0.00 -> 20.9 mm
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